Commit message: Final commit

File: freightRobot/freight_robot_w_camera.gazebo.xacro (robot description, xacro)
@@ -71,8 +71,11 @@
     </sensor>
   </gazebo>
-  <xacro:kinect_ros>
-    <origin xyz="0 0 0.5" rpy="0 -1.60 0" />
-    <inertia ixx="0.1" ixy="0" ixz="0" iyy="0.1" iyz="0" izz="0.1" />
-  </xacro:kinect_ros>
+<gazebo reference="kinect_depth_frame">
+	<sensor type="kinect_ros" name = "depth_camera">
+		<pose>0 0 0 0 0 0</pose>
+		<visualize>true</visualize>
+		<update_rate>15</update_rate>
+	</sensor>
+</gazebo>
   <!-- Color the estop -->
   <gazebo reference="estop_link">
